File: kicad/FC-MAGICON.kicad_sch (KiCad schematic)
At the start: 39 parts, among them J1 Famicom cart edge 60p, J2 LINE OUT 3.5mm, J3 SWD, J4 Cart breakout 2x30, J5 Debug 2x8, J6 USB spare land, P1 Core2350B P1, P2 Core2350B P2, P3 Core2350B P3, P4 Core2350B P4, Q1 2SC1815, SW1 BOOTSEL, SW2 RESET, U2 74LVC245 (5V->3.3V)

Commit message: rev0.2: routed 2-layer board (DRC clean), USB spare land J6, trimmer VR1 for expansion audio, wider power/audio traces, gerbers, 3D images, updated spec
Co-Authored-By: Claude Opus 5.5 <noreply@anthropic.com>
Connections:
- net GND: now also J5.13
- net Q1_B: no longer J5.13
