File: kicad/FC-MAGICON.kicad_pcb (KiCad board)
At the start: 2 copper layers, 90 x 65.8 mm, 39 parts, among them J1 Famicom cart edge 60p, J2 LINE OUT 3.5mm, J3 SWD, J4 Cart breakout 2x30, J5 Debug 2x8, J6 USB spare land, P1 Core2350B P1, P2 Core2350B P2, P3 Core2350B P3, P4 Core2350B P4, Q1 2SC1815, SW1 BOOTSEL, SW2 RESET, U2 74LVC245 (5V->3.3V)

Commit message: rev0.2: routed 2-layer board (DRC clean), USB spare land J6, trimmer VR1 for expansion audio, wider power/audio traces, gerbers, 3D images, updated spec
Co-Authored-By: Claude Opus 5.5 <noreply@anthropic.com>
Connections:
- J5 pad 13: /Q1_B -> /GND
Routing:
- net /GND: track 0.00 -> 338.7 mm, vias 0 -> 134
- net /+5V: track 0.00 -> 151.5 mm, vias 0 -> 2
- net /VBUS_MOD: track 0.00 -> 106.4 mm
- net /EXP_AUDIO_PWM: track 0.00 -> 95.7 mm, vias 0 -> 2
- net /EXP_AUDIO_RC: track 0.00 -> 94.3 mm, vias 0 -> 5
- net /CIRAM_A10: track 0.00 -> 93.5 mm, vias 0 -> 2
- net /+3V3: track 0.00 -> 87.4 mm
- net /IRQ_DRV: track 0.00 -> 87.2 mm, vias 0 -> 2
- net /M2: track 0.00 -> 86.9 mm, vias 0 -> 2
- net /~{IRQ}: track 0.00 -> 80.9 mm, vias 0 -> 6
- net /FC_5V_SENSE: track 0.00 -> 80.1 mm, vias 0 -> 2
- net /CPU_D6: track 0.00 -> 75.5 mm, vias 0 -> 3
- net /SOUND_OUT: track 0.00 -> 72.9 mm, vias 0 -> 2
- net /SOUND_IN: track 0.00 -> 71.0 mm, vias 0 -> 2
- net /PPU_~{A13}: track 0.00 -> 70.8 mm, vias 0 -> 2
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- added copper zone on B.Cu, net /GND
- added copper zone on F.Cu, net /GND
Other:
- board text added: "FC-MAGICON rev0.2"
- board text removed: "FC-MAGICON rev0.1"

Commit message: Back silkscreen: logo, MADE BY SHIMA-R7, spec table; regenerate gerbers/STEP
Co-Authored-By: Claude Opus 5.5 <noreply@anthropic.com>
Other:
- board text added: "CPU A0-14 D0-7"
- board text added: "DBG SWD J3"
- board text added: "MADE BY SHIMA-R7"
- board text added: "MCU RP2350B"
- board text added: "MIR JP1-3"
- board text added: "PCB 1.2t 2L"
- board text added: "PPU AD0-7 A8-13"
- board text added: "RAM 2MB PSRAM"
- board text added: "SND EXP -> 46"
- board text added: "SPEC"
- board text added: "USB FPC / J6"

Commit message: Mount R1 on the back so Q1 can lie down; front silk logo
Co-Authored-By: Claude Opus 5.5 <noreply@anthropic.com>
Parts:
- R1: moved to B.Cu
Other:
- board text added: "rev0.2"
- board text removed: "FC-MAGICON rev0.2"
